File: remote/ib4.sch (KiCad schematic (older format))
At the start: 15 parts, among them J1 Conn_01x02_Female, J2 Screw_Terminal_01x02, J3 Conn_01x07_Female, J6 Screw_Terminal_01x03, J7 Screw_Terminal_01x03, J8 Screw_Terminal_01x03, U2 tpl5110, U3 lora_breakout

Commit message: update
Parts:
- added J4: Conn_01x05_Female, Connector_PinSocket_2.54mm:PinSocket_1x05_P2.54mm_Vertical, symbol Connector:Conn_01x05_Female
- JP2, JP4: footprint ib4:1X14_ROUND70 -> Connector_PinSocket_2.54mm:PinSocket_1x14_P2.54mm_Vertical
- R3: footprint Resistor_THT:R_Axial_DIN0309_L9.0mm_D3.2mm_P5.08mm_Vertical -> Resistor_THT:R_Axial_DIN0411_L9.9mm_D3.6mm_P12.70mm_Horizontal
Connections:
- net labels added: G0
Changed lines of the file:
@@
 F 0 "JP2" H 4150 2725 59  0000 L BNN
 F 1 "HEADER-1X14" H 4150 1100 59  0000 L BNN
-F 2 "ib4:1X14_ROUND70" H 4400 1900 50  0001 C CNN
+F 2 "Connector_PinSocket_2.54mm:PinSocket_1x14_P2.54mm_Vertical" H 4400 1900 50  0001 C CNN
 F 3 "" H 4400 1900 50  0001 C CNN
 	1    4400 1900
@@
 F 0 "JP4" H 7550 2825 59  0000 L BNN
 F 1 "HEADER-1X14" H 7550 1200 59  0000 L BNN
-F 2 "ib4:1X14_ROUND70" H 7800 2000 50  0001 C CNN
+F 2 "Connector_PinSocket_2.54mm:PinSocket_1x14_P2.54mm_Vertical" H 7800 2000 50  0001 C CNN
 F 3 "" H 7800 2000 50  0001 C CNN
 	1    7800 2000
@@
 F 0 "R3" H 4820 4196 50  0000 L CNN
 F 1 "R" H 4820 4105 50  0000 L CNN
-F 2 "Resistor_THT:R_Axial_DIN0309_L9.0mm_D3.2mm_P5.08mm_Vertical" V 4680 4150 50  0001 C CNN
+F 2 "Resistor_THT:R_Axial_DIN0411_L9.9mm_D3.6mm_P12.70mm_Horizontal" V 4680 4150 50  0001 C CNN
 F 3 "~" H 4750 4150 50  0001 C CNN
 	1    4750 4150
@@
 Text GLabel 5350 2950 2    50   Input ~ 0
 TIMED_POWER
+Text GLabel 10050 1800 2    50   Input ~ 0
+G0
+Text GLabel 8300 1900 2    50   Input ~ 0
+G0
+$Comp
+L Connector:Conn_01x05_Female J4
+U 1 1 5E2232E1
+P 11300 1450
+F 0 "J4" H 11328 1476 50  0000 L CNN
+F 1 "Conn_01x05_Female" H 11328 1385 50  0000 L CNN
+F 2 "Connector_PinSocket_2.54mm:PinSocket_1x05_P2.54mm_Vertical" H 11300 1450 50  0001 C CNN
+F 3 "~" H 11300 1450 50  0001 C CNN
+	1    11300 1450
+	1    0    0    -1
+$EndComp
 $EndSCHEMATC
